File: Electrical/KCORES CSPS to ATX Converter/KCORES CSPS to ATX Converter.sch (KiCad schematic (older format))
At the start: 26 parts, among them J1 CSPS, J2 PMBUS, J3 GW_PCIe/CPU, J4 GW_PCIe/CPU, J5 GW_PCIe/CPU, J6 GW_PCIe/CPU, J7 GW_PCIe/CPU, J8 IDE/SATA, J9 GW_24P_ATX, U1 Mini560 5V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

Commit message: Change modules
Used PW22 DC to DC modules instead of defaults
Parts:
- removed U1, U3: Mini560 5V, KCORES_Converter_DCDC:Converter_DCDC_Mini_560, symbol KCORES_Converter_DCDC:Mini560
- removed U2: Mini560 3.3V, KCORES_Converter_DCDC:Converter_DCDC_Mini_560, symbol KCORES_Converter_DCDC:Mini560
- added R5, R6, R7: R, Resistor_SMD:R_0603_1608Metric, symbol Device:R
- added U1, U3: PW22 5V, KCORES_Converter_DCDC:PW22, symbol KCORES_Converter_DCDC:PW22
- added U2: PW22 3.3V, KCORES_Converter_DCDC:PW22, symbol KCORES_Converter_DCDC:PW22
Connections:
- wire segments 314 -> 320

Commit message: Used SMD Packages
Parts:
- C4, C5: footprint Capacitor_THT:C_Disc_D5.0mm_W2.5mm_P2.50mm -> Capacitor_SMD:C_0603_1608Metric
- R1, R2, R3, R4: footprint Resistor_THT:R_Axial_DIN0207_L6.3mm_D2.5mm_P7.62mm_Horizontal -> Resistor_SMD:R_0603_1608Metric
- U4: footprint Package_DIP:DIP-8_W7.62mm -> KCORES_Converter_DCDC:SOIC127P599X175-8N
Changed lines of the file:
@@
 F 0 "R1" V 2293 6250 50  0000 C CNN
 F 1 "22K" V 2384 6250 50  0000 C CNN
-F 2 "Resistor_THT:R_Axial_DIN0207_L6.3mm_D2.5mm_P7.62mm_Horizontal" V 2430 6250 50  0001 C CNN
+F 2 "Resistor_SMD:R_0603_1608Metric" V 2430 6250 50  0001 C CNN
 F 3 "~" H 2500 6250 50  0001 C CNN
 	1    2500 6250
@@
 F 0 "U4" H 7500 7375 50  0000 C CNN
 F 1 "TPS3511" H 7500 7284 50  0000 C CNN
-F 2 "Package_DIP:DIP-8_W7.62mm" H 7500 6750 50  0001 C CNN
+F 2 "KCORES_Converter_DCDC:SOIC127P599X175-8N" H 7500 6750 50  0001 C CNN
 F 3 "" H 8100 6800 50  0001 C CNN
 	1    7500 7000
@@
 F 0 "C4" H 6809 7304 50  0000 R CNN
 F 1 "100nF" H 6809 7395 50  0000 R CNN
-F 2 "Capacitor_THT:C_Disc_D5.0mm_W2.5mm_P2.50mm" H 6900 7350 50  0001 C CNN
+F 2 "Capacitor_SMD:C_0603_1608Metric" H 6900 7350 50  0001 C CNN
 F 3 "~" H 6900 7350 50  0001 C CNN
 	1    6900 7350
@@
 F 0 "R4" H 8191 6654 50  0000 R CNN
 F 1 "3.3K" H 8191 6745 50  0000 R CNN
-F 2 "Resistor_THT:R_Axial_DIN0207_L6.3mm_D2.5mm_P7.62mm_Horizontal" H 8250 6700 50  0001 C CNN
+F 2 "Resistor_SMD:R_0603_1608Metric" H 8250 6700 50  0001 C CNN
 F 3 "~" H 8250 6700 50  0001 C CNN
 	1    8250 6700
@@
 F 0 "C5" H 8092 7396 50  0000 L CNN
 F 1 "100nF" H 8092 7305 50  0000 L CNN
-F 2 "Capacitor_THT:C_Disc_D5.0mm_W2.5mm_P2.50mm" H 8000 7350 50  0001 C CNN
+F 2 "Capacitor_SMD:C_0603_1608Metric" H 8000 7350 50  0001 C CNN
 F 3 "~" H 8000 7350 50  0001 C CNN
 	1    8000 7350
@@
 F 0 "R3" H 6742 6504 50  0000 R CNN
 F 1 "3.3K" H 6742 6595 50  0000 R CNN
-F 2 "Resistor_THT:R_Axial_DIN0207_L6.3mm_D2.5mm_P7.62mm_Horizontal" H 6800 6550 50  0001 C CNN
+F 2 "Resistor_SMD:R_0603_1608Metric" H 6800 6550 50  0001 C CNN
 F 3 "~" H 6800 6550 50  0001 C CNN
 	1    6800 6550
@@
 F 0 "R2" H 6742 6204 50  0000 R CNN
 F 1 "22K" H 6742 6295 50  0000 R CNN
-F 2 "Resistor_THT:R_Axial_DIN0207_L6.3mm_D2.5mm_P7.62mm_Horizontal" H 6800 6250 50  0001 C CNN
+F 2 "Resistor_SMD:R_0603_1608Metric" H 6800 6250 50  0001 C CNN
 F 3 "~" H 6800 6250 50  0001 C CNN
 	1    6800 6250
@@
 ~CSPS_PSON
 $Comp
-L power:+12V #PWR?
+L power:+12V #PWR0101
 U 1 1 60A9F78F
 P 4300 2800
-F 0 "#PWR?" H 4300 2650 50  0001 C CNN
+F 0 "#PWR0101" H 4300 2650 50  0001 C CNN
 F 1 "+12V" H 4315 2973 50  0000 C CNN
 F 2 "" H 4300 2800 50  0001 C CNN
@@
 $EndComp
 $Comp
-L power:GND #PWR?
+L power:GND #PWR0102
 U 1 1 60AFC534
 P 4100 2650
-F 0 "#PWR?" H 4100 2400 50  0001 C CNN
+F 0 "#PWR0102" H 4100 2400 50  0001 C CNN
 F 1 "GND" H 4105 2477 50  0000 C CNN
 F 2 "" H 4100 2650 50  0001 C CNN
@@
 	4100 2550 4300 2550
 $Comp
-L power:+5V #PWR?
+L power:+5V #PWR0103
 U 1 1 60B2A73B
 P 4300 2100
-F 0 "#PWR?" H 4300 1950 50  0001 C CNN
+F 0 "#PWR0103" H 4300 1950 50  0001 C CNN
 F 1 "+5V" H 4315 2273 50  0000 C CNN
 F 2 "" H 4300 2100 50  0001 C CNN
@@
 	5350 2700 5450 2700
 $Comp
-L power:+12V #PWR?
+L power:+12V #PWR0104
 U 1 1 60C78EF3
 P 4300 3900
-F 0 "#PWR?" H 4300 3750 50  0001 C CNN
+F 0 "#PWR0104" H 4300 3750 50  0001 C CNN
 F 1 "+12V" H 4315 4073 50  0000 C CNN
 F 2 "" H 4300 3900 50  0001 C CNN
@@
 $EndComp
 $Comp
-L power:GND #PWR?
+L power:GND #PWR0105
 U 1 1 60C78EFF
 P 4100 3750
-F 0 "#PWR?" H 4100 3500 50  0001 C CNN
+F 0 "#PWR0105" H 4100 3500 50  0001 C CNN
 F 1 "GND" H 4105 3577 50  0000 C CNN
 F 2 "" H 4100 3750 50  0001 C CNN
@@
 	5350 3800 5450 3800
 $Comp
-L power:GND #PWR?
+L power:GND #PWR0106
 U 1 1 60C9523A
 P 4100 5050
-F 0 "#PWR?" H 4100 4800 50  0001 C CNN
+F 0 "#PWR0106" H 4100 4800 50  0001 C CNN
 F 1 "GND" H 4105 4877 50  0000 C CNN
 F 2 "" H 4100 5050 50  0001 C CNN
@@
 	5350 5100 5450 5100
 $Comp
-L power:+3V3 #PWR?
+L power:+3V3 #PWR0107
 U 1 1 60CC977D
 P 4300 3250
-F 0 "#PWR?" H 4300 3100 50  0001 C CNN
+F 0 "#PWR0107" H 4300 3100 50  0001 C CNN
 F 1 "+3V3" H 4315 3423 50  0000 C CNN
 F 2 "" H 4300 3250 50  0001 C CNN

Commit message: csps part
Parts:
- removed C1, C2, C3: 100uF, Capacitor_Tantalum_SMD:CP_EIA-7343-31_Kemet-D_Pad2.25x2.55mm_HandSolder, symbol Device:CP
- removed C4, C5: 100nF, Capacitor_SMD:C_0603_1608Metric, symbol Device:C_Small
- removed D1, D2: 1N4001, Diode_THT:D_DO-41_SOD81_P7.62mm_Horizontal, symbol Device:D_Small
- removed J7: GW_PCIe/CPU, KCORES_Connector_ATX_Power:ATX_8Pin_P4.20mm_Vertical_4.20mm, symbol Connector_Generic:Conn_02x04_Top_Bottom
- removed J8: IDE/SATA, KCORES_Connector_ATX_Power:ATX_4Pin_P4.20mm_Vertical_4.20mm, symbol Connector_Generic:Conn_02x02_Top_Bottom
- removed J9: GW_24P_ATX, KCORES_Connector_ATX_Power:ATX_24Pin_P4.20mm_Vertical_4.20mm, symbol Connector_Generic:Conn_02x12_Top_Bottom
- removed JP1: FPO-CSPS_PSON, Jumper:SolderJumper-2_P1.3mm_Bridged_RoundedPad1.0x1.5mm, symbol Jumper:SolderJumper_2_Bridged
- removed JP2: ATX_PSON-CSPS_PSON, Jumper:SolderJumper-2_P1.3mm_Open_RoundedPad1.0x1.5mm, symbol Jumper:SolderJumper_2_Open
- removed R2: 22K, Resistor_SMD:R_0603_1608Metric, symbol Device:R_Small
- removed R3, R4: 3.3K, Resistor_SMD:R_0603_1608Metric, symbol Device:R_Small
- removed R5, R6, R7: R, Resistor_SMD:R_0603_1608Metric, symbol Device:R
- removed U1, U3: PW22 5V, KCORES_Converter_DCDC:PW22, symbol KCORES_Converter_DCDC:PW22
- removed U2: PW22 3.3V, KCORES_Converter_DCDC:PW22, symbol KCORES_Converter_DCDC:PW22
- removed U4: TPS3511, KCORES_Converter_DCDC:SOIC127P599X175-8N, symbol KCORES_Power_Supervisor:TPS3511
- added SW1: SW_DIP_x01, Button_Switch_THT:SW_DIP_SPSTx01_Slide_9.78x4.72mm_W7.62mm_P2.54mm, symbol Switch:SW_DIP_x01
Connections:
- net +12V: now also J3.5 (Pin_5), J3.6 (Pin_6), J3.7 (Pin_7), J3.8 (Pin_8), J5.5 (Pin_5), J5.6 (Pin_6), J5.7 (Pin_7), J5.8 (Pin_8); no longer J4.1 (Pin_1), J4.2 (Pin_2), J4.3 (Pin_3), J4.4 (Pin_4), J6.1 (Pin_1), J6.2 (Pin_2), J6.3 (Pin_3), J6.4 (Pin_4)
- net GND: now also J4.1 (Pin_1), J4.2 (Pin_2), J4.3 (Pin_3), J4.4 (Pin_4), J6.1 (Pin_1), J6.2 (Pin_2), J6.3 (Pin_3), J6.4 (Pin_4), SW1.2; no longer J3.5 (Pin_5), J3.6 (Pin_6), J3.7 (Pin_7), J3.8 (Pin_8), J5.5 (Pin_5), J5.6 (Pin_6), J5.7 (Pin_7), J5.8 (Pin_8)
- net ~CSPS_PSON: now also SW1.1
- net CSPS_PSOK: no longer names the net of J1.35 (Pin_35)
- no-connect marks 8 -> 6
Other:
- note removed: "1.57V"
- note removed: "JP1 First\nWhen fails, try JP2"
- note removed: "Optional"
- note removed: "U4 Replaceable:\nTPS3510\nTPS3511\nTPS5510\nPS113\nPS113A\nWT7502\nWT7510"

Commit message: v0.1
Parts:
- added M1, M2, M3: Fan_3pin, Connector:FanPinHeader_1x03_P2.54mm_Vertical, symbol Motor:Fan_3pin
Connections:
- net +12V: now also J4.1 (Pin_1), J4.2 (Pin_2), J4.3 (Pin_3), J4.4 (Pin_4), J6.1 (Pin_1), J6.2 (Pin_2), J6.3 (Pin_3), J6.4 (Pin_4), M1.2 (+), M2.2 (+), M3.2 (+); no longer J3.5 (Pin_5), J3.6 (Pin_6), J3.7 (Pin_7), J3.8 (Pin_8), J5.5 (Pin_5), J5.6 (Pin_6), J5.7 (Pin_7), J5.8 (Pin_8)
- net GND: now also J3.5 (Pin_5), J3.6 (Pin_6), J3.7 (Pin_7), J3.8 (Pin_8), J5.5 (Pin_5), J5.6 (Pin_6), J5.7 (Pin_7), J5.8 (Pin_8), M1.3 (-), M2.3 (-), M3.3 (-); no longer J4.1 (Pin_1), J4.2 (Pin_2), J4.3 (Pin_3), J4.4 (Pin_4), J6.1 (Pin_1), J6.2 (Pin_2), J6.3 (Pin_3), J6.4 (Pin_4)
- no-connect marks 6 -> 9
Changed lines of the file:
@@
 Wire Wire Line
 	8450 3750 8450 3650
-Wire Wire Line
-	8350 3650 8350 3750
 $Comp
 L Connector_Generic:Conn_02x04_Top_Bottom J4
@@
 	1    0    0    -1
 $EndComp
+Wire Wire Line
+	8450 2600 8350 2600
+Wire Wire Line
+	8450 2500 8450 2600
+Connection ~ 8450 2600
+Wire Wire Line
+	8550 2600 8450 2600
+Wire Wire Line
+	8550 2500 8550 2600
+Connection ~ 8550 2600
+Wire Wire Line
+	8650 2600 8550 2600
+Wire Wire Line
+	8350 2600 8350 2500
+Wire Wire Line
+	8650 2000 8650 1900
+Wire Wire Line
+	8650 1900 8550 1900
+Connection ~ 8550 1900
+Wire Wire Line
+	8550 2000 8550 1900
+Wire Wire Line
+	8550 1900 8450 1900
+Wire Wire Line
+	8450 1900 8350 1900
+Connection ~ 8450 1900
+Wire Wire Line
+	8450 2000 8450 1900
+Connection ~ 8350 1900
+Wire Wire Line
+	8350 1900 8350 2000
+$Comp
+L power:+12V #PWR020
+U 1 1 60B0B1ED
+P 8350 1800
+F 0 "#PWR020" H 8350 1650 50  0001 C CNN
+F 1 "+12V" H 8365 1973 50  0000 C CNN
+F 2 "" H 8350 1800 50  0001 C CNN
+F 3 "" H 8350 1800 50  0001 C CNN
+	1    8350 1800
+	1    0    0    -1
+$EndComp
+$Comp
+L Connector_Generic:Conn_02x04_Top_Bottom J3
+U 1 1 60B0B1E3
+P 8450 2200
+F 0 "J3" V 8546 2380 50  0000 L CNN
+F 1 "GW_PCIe/CPU" V 8455 2380 50  0000 L CNN
+F 2 "KCORES_Connector_ATX_Power:ATX_8Pin_P4.20mm_Vertical_4.20mm" H 8450 2200 50  0001 C CNN
+F 3 "~" H 8450 2200 50  0001 C CNN
+	1    8450 2200
+	0    -1   1    0
+$EndComp
+$Comp
+L Switch:SW_DIP_x01 SW1
+U 1 1 61545E62
+P 2800 8250
+F 0 "SW1" H 2800 8517 50  0000 C CNN
+F 1 "SW_DIP_x01" H 2800 8426 50  0000 C CNN
+F 2 "Button_Switch_THT:SW_DIP_SPSTx01_Slide_9.78x4.72mm_W7.62mm_P2.54mm" H 2800 8250 50  0001 C CNN
+F 3 "~" H 2800 8250 50  0001 C CNN
+	1    2800 8250
+	1    0    0    -1
+$EndComp
+Text Label 2500 8250 2    50   ~ 0
+~CSPS_PSON
+$Comp
+L power:GND #PWR0101
+U 1 1 61545E69
+P 3100 8250
+F 0 "#PWR0101" H 3100 8000 50  0001 C CNN
+F 1 "GND" H 3105 8077 50  0000 C CNN
+F 2 "" H 3100 8250 50  0001 C CNN
+F 3 "" H 3100 8250 50  0001 C CNN
+	1    3100 8250
+	0    -1   -1   0
+$EndComp
+NoConn ~ 2750 5100
 $Comp
 L Connector_Generic:Conn_02x04_Top_Bottom J5
@@
 	0    -1   1    0
 $EndComp
-Wire Wire Line
-	8450 2600 8350 2600
-Wire Wire Line
-	8450 2500 8450 2600
-Connection ~ 8450 2600
-Wire Wire Line
-	8550 2600 8450 2600
-Wire Wire Line
-	8550 2500 8550 2600
-Connection ~ 8550 2600
-Wire Wire Line
-	8650 2600 8550 2600
-Wire Wire Line
-	8650 2600 8650 2500
-Wire Wire Line
-	8350 2600 8350 2500
-Wire Wire Line
-	8650 2000 8650 1900
-Wire Wire Line
-	8650 1900 8550 1900
-Connection ~ 8550 1900
-Wire Wire Line
-	8550 2000 8550 1900
-Wire Wire Line
-	8550 1900 8450 1900
-Wire Wire Line
-	8450 1900 8350 1900
-Connection ~ 8450 1900
-Wire Wire Line
-	8450 2000 8450 1900
-Connection ~ 8350 1900
-Wire Wire Line
-	8350 1900 8350 2000
-$Comp
-L power:+12V #PWR020
-U 1 1 60B0B1ED
-P 8350 1800
-F 0 "#PWR020" H 8350 1650 50  0001 C CNN
-F 1 "+12V" H 8365 1973 50  0000 C CNN
-F 2 "" H 8350 1800 50  0001 C CNN
-F 3 "" H 8350 1800 50  0001 C CNN
-	1    8350 1800
-	1    0    0    -1
-$EndComp
-$Comp
-L Connector_Generic:Conn_02x04_Top_Bottom J3
-U 1 1 60B0B1E3
-P 8450 2200
-F 0 "J3" V 8546 2380 50  0000 L CNN
-F 1 "GW_PCIe/CPU" V 8455 2380 50  0000 L CNN
-F 2 "KCORES_Connector_ATX_Power:ATX_8Pin_P4.20mm_Vertical_4.20mm" H 8450 2200 50  0001 C CNN
-F 3 "~" H 8450 2200 50  0001 C CNN
-	1    8450 2200
-	0    -1   1    0
-$EndComp
-$Comp
-L Switch:SW_DIP_x01 SW1
-U 1 1 61545E62
-P 2800 8250
-F 0 "SW1" H 2800 8517 50  0000 C CNN
-F 1 "SW_DIP_x01" H 2800 8426 50  0000 C CNN
-F 2 "Button_Switch_THT:SW_DIP_SPSTx01_Slide_9.78x4.72mm_W7.62mm_P2.54mm" H 2800 8250 50  0001 C CNN
-F 3 "~" H 2800 8250 50  0001 C CNN
-	1    2800 8250
-	1    0    0    -1
-$EndComp
-Text Label 2500 8250 2    50   ~ 0
-~CSPS_PSON
-$Comp
-L power:GND #PWR0101
-U 1 1 61545E69
-P 3100 8250
-F 0 "#PWR0101" H 3100 8000 50  0001 C CNN
-F 1 "GND" H 3105 8077 50  0000 C CNN
-F 2 "" H 3100 8250 50  0001 C CNN
-F 3 "" H 3100 8250 50  0001 C CNN
-	1    3100 8250
-	0    -1   -1   0
-$EndComp
-Wire Wire Line
-	10150 3650 10250 3650
-Wire Wire Line
-	10250 3650 10250 4350
-Wire Wire Line
-	10250 4350 10150 4350
-Connection ~ 10150 3650
-Wire Wire Line
-	8650 3650 8750 3650
-Wire Wire Line
-	8750 3650 8750 4350
-Wire Wire Line
-	8750 4350 8650 4350
-Connection ~ 8650 3650
-Wire Wire Line
-	8650 1900 8750 1900
-Wire Wire Line
-	8750 1900 8750 2600
-Wire Wire Line
-	8750 2600 8650 2600
-Connection ~ 8650 1900
+$Comp
+L power:+12V #PWR08
+U 1 1 6152719E
+P 8350 3500
+F 0 "#PWR08" H 8350 3350 50  0001 C CNN
+F 1 "+12V" H 8365 3673 50  0000 C CNN
+F 2 "" H 8350 3500 50  0001 C CNN
+F 3 "" H 8350 3500 50  0001 C CNN
+	1    8350 3500
+	1    0    0    -1
+$EndComp
+Wire Wire Line
+	8350 3500 8350 3650
+Wire Wire Line
+	8350 3750 8350 3650
+Connection ~ 8350 3650
+Wire Wire Line
+	9850 3650 9850 3550
+$Comp
+L power:+12V #PWR010
+U 1 1 6153F2F5
+P 9850 3550
+F 0 "#PWR010" H 9850 3400 50  0001 C CNN
+F 1 "+12V" H 9865 3723 50  0000 C CNN
+F 2 "" H 9850 3550 50  0001 C CNN
+F 3 "" H 9850 3550 50  0001 C CNN
+	1    9850 3550
+	1    0    0    -1
+$EndComp
+$Comp
+L power:GND #PWR09
+U 1 1 61555C12
+P 8650 2750
+F 0 "#PWR09" H 8650 2500 50  0001 C CNN
+F 1 "GND" H 8655 2577 50  0000 C CNN
+F 2 "" H 8650 2750 50  0001 C CNN
+F 3 "" H 8650 2750 50  0001 C CNN
+	1    8650 2750
+	1    0    0    -1
+$EndComp
+Wire Wire Line
+	8650 2600 8650 2750
+Wire Wire Line
+	10150 2700 10150 2600
+$Comp
+L power:GND #PWR011
+U 1 1 6155D239
+P 10150 2700
+F 0 "#PWR011" H 10150 2450 50  0001 C CNN
+F 1 "GND" H 10155 2527 50  0000 C CNN
+F 2 "" H 10150 2700 50  0001 C CNN
+F 3 "" H 10150 2700 50  0001 C CNN
+	1    10150 2700
+	1    0    0    -1
+$EndComp
+Wire Wire Line
+	8650 2500 8650 2600
 Connection ~ 8650 2600
-Wire Wire Line
-	10150 1900 10250 1900
-Wire Wire Line
-	10250 1900 10250 2600
-Wire Wire Line
-	10250 2600 10150 2600
-Connection ~ 10150 1900
-Connection ~ 10150 2600
-NoConn ~ 2750 5100
+$Comp
+L Motor:Fan_3pin M3
+U 1 1 61573953
+P 6400 2100
+F 0 "M3" H 6558 2096 50  0000 L CNN
+F 1 "Fan_3pin" H 6558 2005 50  0000 L CNN
+F 2 "Connector:FanPinHeader_1x03_P2.54mm_Vertical" H 6400 2010 50  0001 C CNN
+F 3 "http://www.hardwarecanucks.com/forum/attachments/new-builds/16287d1330775095-help-chassis-power-fan-connectors-motherboard-asus_p8z68.jpg" H 6400 2010 50  0001 C CNN
+	1    6400 2100
+	1    0    0    -1
+$EndComp
+$Comp
+L Motor:Fan_3pin M2
+U 1 1 61577A46
+P 5550 2100
+F 0 "M2" H 5708 2096 50  0000 L CNN
+F 1 "Fan_3pin" H 5708 2005 50  0000 L CNN
+F 2 "Connector:FanPinHeader_1x03_P2.54mm_Vertical" H 5550 2010 50  0001 C CNN
+F 3 "http://www.hardwarecanucks.com/forum/attachments/new-builds/16287d1330775095-help-chassis-power-fan-connectors-motherboard-asus_p8z68.jpg" H 5550 2010 50  0001 C CNN
+	1    5550 2100
+	1    0    0    -1
+$EndComp
+$Comp
+L Motor:Fan_3pin M1
+U 1 1 6157F715
+P 4800 2100
+F 0 "M1" H 4958 2096 50  0000 L CNN
+F 1 "Fan_3pin" H 4958 2005 50  0000 L CNN
+F 2 "Connector:FanPinHeader_1x03_P2.54mm_Vertical" H 4800 2010 50  0001 C CNN
+F 3 "http://www.hardwarecanucks.com/forum/attachments/new-builds/16287d1330775095-help-chassis-power-fan-connectors-motherboard-asus_p8z68.jpg" H 4800 2010 50  0001 C CNN
+	1    4800 2100
+	1    0    0    -1
+$EndComp
+NoConn ~ 5250 2100
+NoConn ~ 6100 2100
+NoConn ~ 4500 2100
+Wire Wire Line
+	6400 1900 5550 1900
+Connection ~ 5550 1900
+Wire Wire Line
+	5550 1900 4800 1900
+Wire Wire Line
+	6400 2400 5550 2400
+Connection ~ 5550 2400
+Wire Wire Line
+	5550 2400 4800 2400
+Wire Wire Line
+	4800 1900 4800 1800
+$Comp
+L power:+12V #PWR06
+U 1 1 615C66B7
+P 4800 1800
+F 0 "#PWR06" H 4800 1650 50  0001 C CNN
+F 1 "+12V" H 4815 1973 50  0000 C CNN
+F 2 "" H 4800 1800 50  0001 C CNN
+F 3 "" H 4800 1800 50  0001 C CNN
+	1    4800 1800
+	1    0    0    -1
+$EndComp
+$Comp
+L power:GND #PWR07
+U 1 1 615CE608
+P 6400 2550
+F 0 "#PWR07" H 6400 2300 50  0001 C CNN
+F 1 "GND" H 6405 2377 50  0000 C CNN
+F 2 "" H 6400 2550 50  0001 C CNN
+F 3 "" H 6400 2550 50  0001 C CNN
+	1    6400 2550
+	1    0    0    -1
+$EndComp
+Wire Wire Line
+	6400 2400 6400 2550
 $EndSCHEMATC
